File: hardware/eagle/esp_dev_board/dev board.sch (EAGLE design)
At the start: 12 parts, among them U1 TPS7333QD

Commit message: Update schematic
Parts:
- removed JP1, JP2: (no value), pinhead:PINHD-1X8
- removed JP3: (no value), pinhead:PINHD-1X5
- added IC1: INA122P, burr-brown:INA122P
- added LOAD_CELL: 22-23-2041, con-molex:22-23-2041
- added R3, R4: 10k, resistor:R-US_0204/5
- added SV1: USB_TTL, con-lsta:FE05W
- R1: value 10k -> 100
- S1: value Reset -> Config
- S2: value Flash -> Reset
- S3: value (none) -> Flash; device adafruit:EG1218S -> switch-omron:10-XX
Connections:
- removed net 3.3V_REG: C2.1, S3.O, U1.OUT, U1.OUT_2, U1.SENSE/FB
- removed net 3.3V_UART: JP3.1, S3.S
- removed net CH_PD: ESP1.CH_PD, JP1.3, R2.1
- removed net GPIO12: ESP1.GPIO12, JP1.6
- removed net GPIO13: ESP1.GPIO13, JP1.7
- removed net GPIO14: ESP1.GPIO14, JP1.5
- removed net GPIO16: ESP1.GPIO16, JP1.4
- removed net GPIO4: ESP1.GPIO4, JP2.3
- removed net GPIO5: ESP1.GPIO5, JP2.4
- new net N$1: ESP1.CH_PD, R3.1
- new net N$2: IC1.-IN, R1.1
- new net N$3: IC1.RG@1, R1.2
- new net N$4: ESP1.GPIO13, R2.1, S1.P
- new net S+: IC1.+IN, LOAD_CELL-4.S
- new net S-: IC1.RG, LOAD_CELL-3.S
- net 5V_EXT: now also SV1.3; no longer JP3.3
- net ADC: now also IC1.OUT; no longer JP1.2
- net GND: now also IC1.REF, IC1.V-, LOAD_CELL-1.S, S1.S1, S2.P1, S3.S1, SV1.4; no longer JP2.7, JP2.8, JP3.2, S1.P1, S2.S1
- net GPIO0: now also S3.P1; no longer JP2.5, S2.P1
- net RST: now also R4.1, S2.S; no longer JP1.1, R1.1, S1.S
- net RX: now also SV1.2; no longer JP2.2, JP3.4
- net TX: now also SV1.1; no longer JP2.1, JP3.5
- net VCC: now also C2.1, IC1.V+, LOAD_CELL-2.S, R3.2, R4.2, U1.OUT, U1.OUT_2, U1.SENSE/FB; no longer JP1.8, JP2.6, R1.2, S3.P
Other:
- note removed: "Female header"
- moved on the sheet: C1, C2, ESP1, R1, R2, S1, S2, U1
